File: PCH-1000JIG ALT/Kicad/PCH-1000JIG.kicad_pcb (KiCad board)
At the start: 2 copper layers, 73.7 x 61 mm, 14 parts

Commit message: Added version 1.3 if the throughhole board
Changed BOM to use one less resistor
Siplified board
Added an ALT design to use the previous (possibly more reliable) resistor values.
Parts:
- added 330 Ohms: R_Axial_DIN0309_L9.0mm_D3.2mm_P12.70mm_Horizontal, Resistor_THT:R_Axial_DIN0309_L9.0mm_D3.2mm_P12.70mm_Horizontal, F.Cu at (48.3, 36.4)
- 150 Ohms: renamed from 220 Ohms
- 330 Ohms: renamed from 1k Ohms
Routing:
- net (no net): track 532.8 -> 530.0 mm
Other:
- board text added: "PCH-1000 JIG BOARD 1.3 ALT By Mathieulh"
- board text removed: "PCH-1000 JIG BOARD 1.3 By Mathieulh"
Changed lines of the file:
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@@
     (tags "Resistor Axial_DIN0309 series Axial Horizontal pin pitch 12.7mm 0.5W = 1/2W length 9mm diameter 3.2mm")
     (attr through_hole)
-    (fp_text reference "1k Ohms" (at 6.35 -2.72) (layer "F.SilkS")
+    (fp_text reference "330 Ohms" (at 6.35 -2.72) (layer "F.SilkS")
         (effects (font (size 1 1) (thickness 0.15)))
     )
@@
     (pad "1" smd circle (at 0 0) (size 2 2) (layers "F.Cu" "F.Mask"))
   )
+  (footprint "Resistor_THT:R_Axial_DIN0309_L9.0mm_D3.2mm_P12.70mm_Horizontal" (layer "F.Cu")
+    (at 48.26 36.38)
+    (descr "Resistor, Axial_DIN0309 series, Axial, Horizontal, pin pitch=12.7mm, 0.5W = 1/2W, length*diameter=9*3.2mm^2, http://cdn-reichelt.de/documents/datenblatt/B400/1_4W%23YAG.pdf")
+    (tags "Resistor Axial_DIN0309 series Axial Horizontal pin pitch 12.7mm 0.5W = 1/2W length 9mm diameter 3.2mm")
+    (attr through_hole)
+    (fp_text reference "330 Ohms" (at 6.35 -2.72) (layer "F.SilkS")
+        (effects (font (size 1 1) (thickness 0.15)))
+    )
+    (fp_text value "R_Axial_DIN0309_L9.0mm_D3.2mm_P12.70mm_Horizontal" (at 6.35 2.72) (layer "F.Fab")
+        (effects (font (size 1 1) (thickness 0.15)))
+    )
+    (fp_text user "${REFERENCE}" (at 6.35 0) (layer "F.Fab")
+        (effects (font (size 1 1) (thickness 0.15)))
+    )
+    (fp_line (start 1.04 0) (end 1.73 0)
+      (stroke (width 0.12) (type solid)) (layer "F.SilkS"))
+    (fp_line (start 1.73 -1.72) (end 1.73 1.72)
+      (stroke (width 0.12) (type solid)) (layer "F.SilkS"))
+    (fp_line (start 1.73 1.72) (end 10.97 1.72)
+      (stroke (width 0.12) (type solid)) (layer "F.SilkS"))
+    (fp_line (start 10.97 -1.72) (end 1.73 -1.72)
+      (stroke (width 0.12) (type solid)) (layer "F.SilkS"))
+    (fp_line (start 10.97 1.72) (end 10.97 -1.72)
+      (stroke (width 0.12) (type solid)) (layer "F.SilkS"))
+    (fp_line (start 11.66 0) (end 10.97 0)
+      (stroke (width 0.12) (type solid)) (layer "F.SilkS"))
+    (fp_line (start -1.05 -1.85) (end -1.05 1.85)
+      (stroke (width 0.05) (type solid)) (layer "F.CrtYd"))
+    (fp_line (start -1.05 1.85) (end 13.75 1.85)
+      (stroke (width 0.05) (type solid)) (layer "F.CrtYd"))
+    (fp_line (start 13.75 -1.85) (end -1.05 -1.85)
+      (stroke (width 0.05) (type solid)) (layer "F.CrtYd"))
+    (fp_line (start 13.75 1.85) (end 13.75 -1.85)
+      (stroke (width 0.05) (type solid)) (layer "F.CrtYd"))
+    (fp_line (start 0 0) (end 1.85 0)
+      (stroke (width 0.1) (type solid)) (layer "F.Fab"))
+    (fp_line (start 1.85 -1.6) (end 1.85 1.6)
+      (stroke (width 0.1) (type solid)) (layer "F.Fab"))
+    (fp_line (start 1.85 1.6) (end 10.85 1.6)
+      (stroke (width 0.1) (type solid)) (layer "F.Fab"))
+    (fp_line (start 10.85 -1.6) (end 1.85 -1.6)
+      (stroke (width 0.1) (type solid)) (layer "F.Fab"))
+    (fp_line (start 10.85 1.6) (end 10.85 -1.6)
+      (stroke (width 0.1) (type solid)) (layer "F.Fab"))
+    (fp_line (start 12.7 0) (end 10.85 0)
+      (stroke (width 0.1) (type solid)) (layer "F.Fab"))
+    (pad "1" thru_hole circle (at 0 0) (size 1.6 1.6) (drill 0.8) (layers "*.Cu" "*.Mask"))
+    (pad "2" thru_hole oval (at 12.7 0) (size 1.6 1.6) (drill 0.8) (layers "*.Cu" "*.Mask"))
+    (model "${KICAD6_3DMODEL_DIR}/Resistor_THT.3dshapes/R_Axial_DIN0309_L9.0mm_D3.2mm_P12.70mm_Horizontal.wrl"
+      (offset (xyz 0 0 0))
+      (scale (xyz 1 1 1))
+      (rotate (xyz 0 0 0))
+    )
+  )
   (footprint "TestPoint:TestPoint_Pad_D2.0mm" (layer "F.Cu")
     (at 48.26 51.62)
@@
     (tags "Resistor Axial_DIN0309 series Axial Horizontal pin pitch 12.7mm 0.5W = 1/2W length 9mm diameter 3.2mm")
     (attr through_hole)
-    (fp_text reference "220 Ohms" (at 6.35 -2.72) (layer "F.SilkS")
+    (fp_text reference "150 Ohms" (at 6.35 -2.72) (layer "F.SilkS")
         (effects (font (size 1 1) (thickness 0.15)))
     )
@@
   (gr_rect (start 20.32 13.52) (end 93.98 74.48)
     (stroke (width 0.1) (type default)) (fill none) (layer "Edge.Cuts"))
-  (gr_text "PCH-1000 JIG BOARD 1.3\nBy Mathieulh" (at 60.96 30.48) (layer "F.SilkS")
+  (gr_text "PCH-1000 JIG BOARD 1.3 ALT\nBy Mathieulh" (at 58.42 30.48) (layer "F.SilkS")
     (effects (font (size 1.5 1.5) (thickness 0.3) bold) (justify left bottom))
   )
+  (segment (start 67.76 36.38) (end 67.76 44.9) (width 0.25) (layer "F.Cu") (net 0))
   (segment (start 40.64 51.62) (end 45.72 46.54) (width 0.25) (layer "F.Cu") (net 0))
   (segment (start 58.42 21.14) (end 60.96 21.14) (width 0.25) (layer "F.Cu") (net 0))
@@
   (segment (start 60.96 36.38) (end 67.76 36.38) (width 0.25) (layer "F.Cu") (net 0))
   (segment (start 25.4 59.24) (end 22.985 61.655) (width 0.25) (layer "F.Cu") (net 0))
+  (segment (start 67.76 44.9) (end 71.12 48.26) (width 0.25) (layer "F.Cu") (net 0))
   (segment (start 45.72 54.16) (end 48.26 51.62) (width 0.25) (layer "F.Cu") (net 0))
   (segment (start 45.72 33.84) (end 58.42 21.14) (width 0.25) (layer "F.Cu") (net 0))
@@
   (segment (start 83.82 36.38) (end 83.82 49.08) (width 0.25) (layer "F.Cu") (net 0))
   (segment (start 63.5 56.7) (end 63.5 51.62) (width 0.25) (layer "F.Cu") (net 0))
-  (segment (start 71.12 51.62) (end 71.12 46.54) (width 0.25) (layer "F.Cu") (net 0))
   (segment (start 63.5 46.54) (end 63.5 51.62) (width 0.25) (layer "F.Cu") (net 0))
   (segment (start 71.12 56.7) (end 71.12 51.62) (width 0.25) (layer "F.Cu") (net 0))
-  (segment (start 71.12 46.54) (end 60.96 36.38) (width 0.25) (layer "F.Cu") (net 0))
   (segment (start 33.02 51.62) (end 33.02 21.14) (width 0.25) (layer "F.Cu") (net 0))
   (segment (start 33.02 21.14) (end 26.67 21.14) (width 0.25) (layer "F.Cu") (net 0))
   (segment (start 86.36 51.62) (end 86.36 61.78) (width 0.25) (layer "F.Cu") (net 0))
+  (segment (start 71.12 51.62) (end 71.12 48.26) (width 0.25) (layer "F.Cu") (net 0))
   (segment (start 30.48 59.24) (end 38.1 51.62) (width 0.25) (layer "F.Cu") (net 0))
   (segment (start 31.4 61.78) (end 29.4 61.78) (width 0.25) (layer "F.Cu") (net 0))
